File: Z80_Debugger.kicad_sch (KiCad schematic)
At the start: 35 parts, among them J1 ICSP, J2 UART, J3 I2C, J4 microSD, J6 M1_O, J7 USB_B_Mini, U1 Z84C00_PLCC, U2 PIC18F4520-xP, U3 AS6C4008-55PCN, U4 74HC138, U5 74AHC273, U6 74HC595, U7 74HC595, U8 74HC595, Y1 CXO_DIP8, Y2 Crystal

Commit message: add pins: M1, RD, WR for Z80 Req
Parts:
- removed J6: M1_O, Connector_PinHeader_2.54mm:PinHeader_1x01_P2.54mm_Vertical, symbol Connector_Generic:Conn_01x01
Connections:
- net 0x81: now also U2.9 (RE1); no longer U2.4 (RA2)
- net 0x82: no longer U2.5 (RA3)
- net IORQ: now also U2.7 (RA5)
- net M1: now also U2.4 (RA2)
- net RD: now also U2.5 (RA3)
- net WR: now also U2.6 (RA4); no longer U2.9 (RE1)
- net 0x83: no longer names the net of U4.12 (~{Y3})
- net 0x83: no longer U2.6 (RA4)
- net 0x84: no longer names the net of U4.11 (~{Y4})
- net 0x84: no longer U2.7 (RA5)
- no-connect marks 21 -> 23
Other:
- note added: "Wait M1 + IORQ = LOW And RD + WR = HIGH To Z80 Request."
- note removed: "Let anything observe CPU Instruction Fetch"
Changed lines of the file:
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@@
 		)
 	)
-	(text "Need Pull-UP HIGH : \nPrevents Z80 glitching during \nPIC power-on boot phase."
+	(text "Wait M1 + IORQ = LOW\nAnd RD + WR = HIGH\nTo Z80 Request."
 		(exclude_from_sim no)
-		(at 16.51 136.398 0)
+		(at 214.63 48.006 0)
 		(effects
 			(font
@@
 		)
 	)
-	(text "Need to PUll-UP HIGH,\nAs Active-Low to disable.\nAS6C4008 is 55ns too fast to wait."
+	(text "Need Pull-UP HIGH : \nPrevents Z80 glitching during \nPIC power-on boot phase."
 		(exclude_from_sim no)
-		(at 16.256 113.284 0)
+		(at 16.51 136.398 0)
 		(effects
 			(font
@@
 		)
 	)
-	(text "Need Pull-UP HIGH : \nKeeps Z80 running normally \nuntil PIC requests the bus."
+	(text "Need to PUll-UP HIGH,\nAs Active-Low to disable.\nAS6C4008 is 55ns too fast to wait."
 		(exclude_from_sim no)
-		(at 16.256 128.778 0)
+		(at 16.256 113.284 0)
 		(effects
 			(font
@@
 		)
 	)
-	(text "Pull BUSREQ -> LOW to force\nZ80 release Address Bus\nand copy ROM from \nmicroSD -> SRAM"
+	(text "Need Pull-UP HIGH : \nKeeps Z80 running normally \nuntil PIC requests the bus."
 		(exclude_from_sim no)
-		(at 210.82 69.088 0)
+		(at 16.256 128.778 0)
 		(effects
 			(font
@@
 		)
 	)
-	(text "Let anything observe \nCPU Instruction Fetch "
+	(text "Pull BUSREQ -> LOW to force\nZ80 release Address Bus\nand copy ROM from \nmicroSD -> SRAM"
 		(exclude_from_sim no)
-		(at 16.256 105.918 0)
+		(at 210.82 69.088 0)
 		(effects
 			(font
@@
 	)
 	(no_connect
+		(at 44.45 170.18)
+	)
+	(no_connect
 		(at 179.07 114.3)
 	)
@@
 	)
 	(no_connect
+		(at 44.45 167.64)
+	)
+	(no_connect
 		(at 179.07 124.46)
 	)
@@
 	(wire
 		(pts
-			(xy 222.25 50.8) (xy 240.03 50.8)
+			(xy 227.33 50.8) (xy 240.03 50.8)
 		)
 		(stroke
@@
 	(wire
 		(pts
+			(xy 227.33 55.88) (xy 240.03 55.88)
+		)
+		(stroke
+			(width 0)
+			(type default)
+		)
+	)
+	(wire
+		(pts
 			(xy 109.22 106.68) (xy 119.38 106.68)
 		)
@@
 	(wire
 		(pts
-			(xy 222.25 55.88) (xy 240.03 55.88)
-		)
-		(stroke
-			(width 0)
-			(type default)
-		)
-	)
-	(wire
-		(pts
 			(xy 201.93 125.73) (xy 198.12 125.73)
 		)
@@
 	(wire
 		(pts
-			(xy 44.45 170.18) (xy 55.88 170.18)
-		)
-		(stroke
-			(width 0)
-			(type default)
-		)
-	)
-	(wire
-		(pts
 			(xy 101.6 20.32) (xy 101.6 24.13)
 		)
@@
 	(wire
 		(pts
-			(xy 44.45 167.64) (xy 55.88 167.64)
-		)
-		(stroke
-			(width 0)
-			(type default)
-		)
-	)
-	(wire
-		(pts
 			(xy 227.33 43.18) (xy 240.03 43.18)
 		)
@@
 	(wire
 		(pts
-			(xy 222.25 53.34) (xy 240.03 53.34)
+			(xy 227.33 53.34) (xy 240.03 53.34)
 		)
 		(stroke
@@
 	(wire
 		(pts
-			(xy 222.25 48.26) (xy 240.03 48.26)
+			(xy 227.33 48.26) (xy 240.03 48.26)
 		)
 		(stroke
@@
 	(wire
 		(pts
-			(xy 16.51 104.14) (xy 30.48 104.14)
-		)
-		(stroke
-			(width 0)
-			(type default)
-		)
-	)
-	(wire
-		(pts
 			(xy 125.73 160.02) (xy 115.57 160.02)
 		)
@@
 		)
 	)
+	(label "0x82"
+		(at 219.71 39.37 0)
+		(effects
+			(font
+				(size 1.27 1.27)
+			)
+			(justify left bottom)
+		)
+	)
 	(label "SCK"
 		(at 281.94 55.88 180)
@@
 		)
 	)
-	(label "WR"
-		(at 227.33 35.56 0)
-		(effects
-			(font
-				(size 1.27 1.27)
-			)
-			(justify left bottom)
-		)
-	)
 	(label "A3"
 		(at 74.93 36.83 180)
@@
 		)
 	)
+	(label "RD"
+		(at 227.33 50.8 0)
+		(effects
+			(font
+				(size 1.27 1.27)
+			)
+			(justify left bottom)
+		)
+	)
 	(label "A16"
 		(at 125.73 154.94 180)
@@
 		)
 	)
-	(label "M1"
-		(at 16.51 104.14 0)
-		(effects
-			(font
-				(size 1.27 1.27)
-			)
-			(justify left bottom)
-		)
-	)
 	(label "WAIT"
 		(at 25.4 54.61 0)
@@
 		)
 	)
-	(label "WR"
-		(at 17.78 175.26 0)
+	(label "IORQ"
+		(at 227.33 55.88 0)
 		(effects
 			(font
@@
 		)
 	)
-	(label "0x84"
-		(at 222.25 55.88 0)
+	(label "WR"
+		(at 17.78 175.26 0)
 		(effects
 			(font
@@
 		)
 	)
-	(label "0x83"
-		(at 222.25 53.34 0)
-		(effects
-			(font
-				(size 1.27 1.27)
-			)
-			(justify left bottom)
-		)
-	)
 	(label "PGD"
 		(at 256.54 132.08 0)
@@
 		)
 	)
+	(label "WR"
+		(at 227.33 53.34 0)
+		(effects
+			(font
+				(size 1.27 1.27)
+			)
+			(justify left bottom)
+		)
+	)
+	(label "0x81"
+		(at 227.33 35.56 0)
+		(effects
+			(font
+				(size 1.27 1.27)
+			)
+			(justify left bottom)
+		)
+	)
 	(label "MCLR"
 		(at 256.54 124.46 0)
@@
 		)
 	)
-	(label "0x82"
-		(at 222.25 50.8 0)
-		(effects
-			(font
-				(size 1.27 1.27)
-			)
-			(justify left bottom)
-		)
-	)
-	(label "0x84"
-		(at 55.88 170.18 180)
+	(label "A14"
+		(at 74.93 64.77 180)
 		(effects
 			(font
@@
 		)
 	)
-	(label "A14"
-		(at 74.93 64.77 180)
+	(label "SRCLK"
+		(at 111.76 111.76 0)
 		(effects
 			(font
 				(size 1.27 1.27)
 			)
-			(justify right bottom)
+			(justify left bottom)
 		)
 	)
-	(label "SRCLK"
-		(at 111.76 111.76 0)
+	(label "M1"
+		(at 227.33 48.26 0)
 		(effects
 			(font
@@
 		)
 	)
-	(label "0x83"
-		(at 55.88 167.64 180)
-		(effects
-			(font
-				(size 1.27 1.27)
-			)
-			(justify right bottom)
-		)
-	)
 	(label "RESET"
 		(at 80.01 180.34 0)
@@
 		)
 	)
-	(label "0x81"
-		(at 222.25 48.26 0)
-		(effects
-			(font
-				(size 1.27 1.27)
-			)
-			(justify left bottom)
-		)
-	)
 	(label "VCC"
 		(at 234.95 153.67 0)
@@
 					(unit 1)
 				)
-			)
-		)
-	)
-	(symbol
-		(lib_id "Connector_Generic:Conn_01x01")
-		(at 35.56 104.14 0)
-		(unit 1)
-		(body_style 1)
-		(exclude_from_sim no)
-		(in_bom yes)
-		(on_board yes)
-		(in_pos_files yes)
-		(dnp no)
-		(fields_autoplaced yes)
-		(property "Reference" "J6"
-			(at 38.1 102.8699 0)
-			(show_name no)
-			(do_not_autoplace no)
-			(effects
-				(font
-					(size 1.27 1.27)
-				)
-				(justify left)
-			)
-		)
-		(property "Value" "M1_O"
-			(at 38.1 105.4099 0)
-			(show_name no)
-			(do_not_autoplace no)
-			(effects
-				(font
-					(size 1.27 1.27)
-				)
-				(justify left)
-			)
-		)
-		(property "Footprint" "Connector_PinHeader_2.54mm:PinHeader_1x01_P2.54mm_Vertical"
-			(at 35.56 104.14 0)
-			(hide yes)
-			(show_name no)
-			(do_not_autoplace no)
-			(effects
-				(font
-					(size 1.27 1.27)
-				)
-			)
-		)
-		(property "Datasheet" ""
-			(at 35.56 104.14 0)
-			(hide yes)
-			(show_name no)
-			(do_not_autoplace no)
-			(effects
-				(font
-					(size 1.27 1.27)
-				)
-			)
-		)
-		(property "Description" "Generic connector, single row, 01x01, script generated (kicad-library-utils/schlib/autogen/connector/)"
-			(at 35.56 104.14 0)
-			(hide yes)
-			(show_name no)
-			(do_not_autoplace no)
-			(effects
-				(font
-					(size 1.27 1.27)
-				)
-			)
-		)
-		(pin "1"
-		)
-		(instances
-			(project "Z80_Debugger"
-				(path "/1dee2e6f-8929-455d-a1de-5fd790cf69ac"
-					(reference "J6")
-					(unit 1)
-				)
